File: Elephant-3/Elephant-3.sch (KiCad schematic (older format))
At the start: 10 parts

Commit message: Made Schemiatic version 1
Parts:
- removed U?: mc34151, Housings_DIP:DIP-8_W7.62mm, symbol mc34151p:mc34151
- added C4D02120, D?: D, symbol device:D
- added C?: C, symbol device:C
- added C? (x2): 22pF, symbol device:C
- added C? (x3): 100nF, symbol device:C
- added C?: 4.7uF, symbol device:CP
- added C? (x4): 10nF, symbol device:C
- added D? (x8): D_Schottky, symbol device:D_Schottky
- added J?: Switch, symbol Connector:Conn_01x02
- added J?: 300V, symbol Connector:Conn_01x02
- added J?: 1200V, symbol Connector:Conn_01x02
- added J?: Ignitor, symbol Connector:Conn_01x02
- added J?: Main, symbol Connector:Conn_01x02
- added J?: 18V, symbol Connector:Conn_01x02
- added J?: ADC2, symbol Connector:Conn_01x03
- added J?: ADC1, symbol Connector:Conn_01x03
- added J?: ADC0, symbol Connector:Conn_01x03
- added J?: IgnCap, symbol Connector:Conn_01x02
- added Q?: IRGPS40B120U, symbol device:Q_NIGBT_GCE
- added Q?: Q_NMOS_GDS, symbol device:Q_NMOS_GDS
- added R? (x3): 10k, symbol device:R
- added R? (x2): 340k, symbol device:R
- added R? (x4): 680, symbol device:R
- added R?: 680k, symbol device:R
- added SW?: Reset, symbol Switch:SW_DIP_x01
- added U?: MC34151, Housings_DIP:DIP-8_W7.62mm, symbol mc34151p:MC34151
- added Y?: 16MHz, symbol device:Crystal
Connections:
- net labels added: 1200V, 18V, 300V, GNDA, IgnCap
- wire segments 33 -> 201

Commit message: few bug fix
Parts:
- Q?: value Q_NMOS_GDS -> STW21N150K5
Connections:
- wire segments 201 -> 200
Changed lines of the file:
@@
 	9050 3350 9050 3700
-Wire Wire Line
-	9150 3150 9150 3250
 Wire Wire Line
 	8750 3550 8750 3700
@@
 P 10150 3150
 F 0 "Q?" H 10355 3196 50  0000 L CNN
-F 1 "Q_NMOS_GDS" H 10355 3105 50  0000 L CNN
+F 1 "STW21N150K5" H 10355 3105 50  0000 L CNN
 F 2 "" H 10350 3250 50  0001 C CNN
 F 3 "" H 10150 3150 50  0001 C CNN

Commit message: Updated capacitor value
Parts:
- C?: value C -> 5uF
Changed lines of the file:
@@
 P 7700 2800
 F 0 "C?" V 7448 2800 50  0000 C CNN
-F 1 "C" V 7539 2800 50  0000 C CNN
+F 1 "5uF" V 7539 2800 50  0000 C CNN
 F 2 "" H 7738 2650 50  0001 C CNN
 F 3 "" H 7700 2800 50  0001 C CNN

Commit message: Wrong placement of capacitor
Connections:
- wire segments 200 -> 202
Changed lines of the file:
@@
 L device:R R?
 U 1 1 5A46F515
-P 3450 6050
-F 0 "R?" H 3520 6096 50  0000 L CNN
-F 1 "680" H 3520 6005 50  0000 L CNN
-F 2 "" V 3380 6050 50  0001 C CNN
-F 3 "" H 3450 6050 50  0001 C CNN
-	1    3450 6050
+P 3450 6450
+F 0 "R?" H 3520 6496 50  0000 L CNN
+F 1 "680" H 3520 6405 50  0000 L CNN
+F 2 "" V 3380 6450 50  0001 C CNN
+F 3 "" H 3450 6450 50  0001 C CNN
+	1    3450 6450
 	1    0    0    -1
 $EndComp
@@
 L device:C C?
 U 1 1 5A46F78A
-P 3250 6350
-F 0 "C?" V 2998 6350 50  0000 C CNN
-F 1 "10nF" V 3089 6350 50  0000 C CNN
-F 2 "" H 3288 6200 50  0001 C CNN
-F 3 "" H 3250 6350 50  0001 C CNN
-	1    3250 6350
+P 3250 6200
+F 0 "C?" V 2998 6200 50  0000 C CNN
+F 1 "10nF" V 3089 6200 50  0000 C CNN
+F 2 "" H 3288 6050 50  0001 C CNN
+F 3 "" H 3250 6200 50  0001 C CNN
+	1    3250 6200
 	0    1    1    0
 $EndComp
 Wire Wire Line
-	3050 6350 3050 6700
+	3050 6200 3050 6700
 Connection ~ 3050 6700
-Wire Wire Line
-	3400 6350 3450 6350
-Wire Wire Line
-	3450 6350 3450 6200
-Wire Wire Line
-	3450 6350 3450 6700
-Connection ~ 3450 6350
 Connection ~ 3450 6700
 Wire Wire Line
 	3450 6700 3500 6700
 Wire Wire Line
-	3050 6350 3100 6350
+	3050 6200 3100 6200
 $Comp
 L device:D_Schottky D?
@@
 L device:R R?
 U 1 1 5A4955F1
-P 4450 6050
-F 0 "R?" H 4520 6096 50  0000 L CNN
-F 1 "680" H 4520 6005 50  0000 L CNN
-F 2 "" V 4380 6050 50  0001 C CNN
-F 3 "" H 4450 6050 50  0001 C CNN
-	1    4450 6050
+P 4450 6450
+F 0 "R?" H 4520 6496 50  0000 L CNN
+F 1 "680" H 4520 6405 50  0000 L CNN
+F 2 "" V 4380 6450 50  0001 C CNN
+F 3 "" H 4450 6450 50  0001 C CNN
+	1    4450 6450
 	1    0    0    -1
 $EndComp
@@
 L device:C C?
 U 1 1 5A4955F8
-P 4250 6350
-F 0 "C?" V 3998 6350 50  0000 C CNN
-F 1 "10nF" V 4089 6350 50  0000 C CNN
-F 2 "" H 4288 6200 50  0001 C CNN
-F 3 "" H 4250 6350 50  0001 C CNN
-	1    4250 6350
+P 4250 6200
+F 0 "C?" V 3998 6200 50  0000 C CNN
+F 1 "10nF" V 4089 6200 50  0000 C CNN
+F 2 "" H 4288 6050 50  0001 C CNN
+F 3 "" H 4250 6200 50  0001 C CNN
+	1    4250 6200
 	0    1    1    0
 $EndComp
 Wire Wire Line
-	4050 6350 4050 6700
+	4050 6200 4050 6700
 Connection ~ 4050 6700
-Wire Wire Line
-	4400 6350 4450 6350
-Wire Wire Line
-	4450 6350 4450 6200
-Wire Wire Line
-	4450 6350 4450 6700
-Connection ~ 4450 6350
 Connection ~ 4450 6700
 Wire Wire Line
 	4450 6700 4500 6700
 Wire Wire Line
-	4050 6350 4100 6350
+	4050 6200 4100 6200
 $Comp
 L device:D_Schottky D?
@@
 L device:R R?
 U 1 1 5A49A313
-P 5450 6050
-F 0 "R?" H 5520 6096 50  0000 L CNN
-F 1 "680" H 5520 6005 50  0000 L CNN
-F 2 "" V 5380 6050 50  0001 C CNN
-F 3 "" H 5450 6050 50  0001 C CNN
-	1    5450 6050
+P 5450 6450
+F 0 "R?" H 5520 6496 50  0000 L CNN
+F 1 "680" H 5520 6405 50  0000 L CNN
+F 2 "" V 5380 6450 50  0001 C CNN
+F 3 "" H 5450 6450 50  0001 C CNN
+	1    5450 6450
 	1    0    0    -1
 $EndComp
@@
 L device:C C?
 U 1 1 5A49A31A
-P 5250 6350
-F 0 "C?" V 4998 6350 50  0000 C CNN
-F 1 "10nF" V 5089 6350 50  0000 C CNN
-F 2 "" H 5288 6200 50  0001 C CNN
-F 3 "" H 5250 6350 50  0001 C CNN
-	1    5250 6350
+P 5250 6200
+F 0 "C?" V 4998 6200 50  0000 C CNN
+F 1 "10nF" V 5089 6200 50  0000 C CNN
+F 2 "" H 5288 6050 50  0001 C CNN
+F 3 "" H 5250 6200 50  0001 C CNN
+	1    5250 6200
 	0    1    1    0
 $EndComp
 Wire Wire Line
-	5050 6350 5050 6700
+	5050 6200 5050 6700
 Connection ~ 5050 6700
-Wire Wire Line
-	5400 6350 5450 6350
-Wire Wire Line
-	5450 6350 5450 6200
-Wire Wire Line
-	5450 6350 5450 6700
-Connection ~ 5450 6350
 Connection ~ 5450 6700
 Wire Wire Line
 	5450 6700 5500 6700
 Wire Wire Line
-	5050 6350 5100 6350
+	5050 6200 5100 6200
 Connection ~ 5200 4650
 Wire Wire Line
@@
 	4000 5900 4000 4000
 Wire Wire Line
-	5450 5900 5450 5800
+	5450 6300 5450 6200
 Wire Wire Line
 	4100 5800 4100 3900
@@
 L device:R R?
 U 1 1 5A85E22D
-P 2450 6050
-F 0 "R?" H 2520 6096 50  0000 L CNN
-F 1 "680" H 2520 6005 50  0000 L CNN
-F 2 "" V 2380 6050 50  0001 C CNN
-F 3 "" H 2450 6050 50  0001 C CNN
-	1    2450 6050
+P 2450 6450
+F 0 "R?" H 2520 6496 50  0000 L CNN
+F 1 "680" H 2520 6405 50  0000 L CNN
+F 2 "" V 2380 6450 50  0001 C CNN
+F 3 "" H 2450 6450 50  0001 C CNN
+	1    2450 6450
 	1    0    0    -1
 $EndComp
@@
 L device:C C?
 U 1 1 5A85E234
-P 2250 6350
-F 0 "C?" V 1998 6350 50  0000 C CNN
-F 1 "10nF" V 2089 6350 50  0000 C CNN
-F 2 "" H 2288 6200 50  0001 C CNN
-F 3 "" H 2250 6350 50  0001 C CNN
-	1    2250 6350
+P 2250 6200
+F 0 "C?" V 1998 6200 50  0000 C CNN
+F 1 "10nF" V 2089 6200 50  0000 C CNN
+F 2 "" H 2288 6050 50  0001 C CNN
+F 3 "" H 2250 6200 50  0001 C CNN
+	1    2250 6200
 	0    1    1    0
 $EndComp
 Wire Wire Line
-	2050 6350 2050 6700
+	2050 6200 2050 6700
 Connection ~ 2050 6700
-Wire Wire Line
-	2400 6350 2450 6350
-Wire Wire Line
-	2450 6350 2450 6200
-Wire Wire Line
-	2450 6350 2450 6700
-Connection ~ 2450 6350
 Connection ~ 2450 6700
 Wire Wire Line
 	2450 6700 2500 6700
 Wire Wire Line
-	2050 6350 2100 6350
-Wire Wire Line
-	2450 7300 2450 6700
+	2050 6200 2100 6200
 Wire Wire Line
 	5450 5800 4100 5800
 Wire Wire Line
-	2450 5900 2450 5800
+	2450 6300 2450 6200
 Wire Wire Line
 	2450 5800 3800 5800
@@
 Wire Wire Line
 	4250 1150 4250 1250
+Wire Wire Line
+	5400 6200 5450 6200
+Connection ~ 5450 6200
+Wire Wire Line
+	5450 6200 5450 5800
+Wire Wire Line
+	5450 6600 5450 6700
+Wire Wire Line
+	4450 6300 4450 6200
+Wire Wire Line
+	4400 6200 4450 6200
+Connection ~ 4450 6200
+Wire Wire Line
+	4450 6200 4450 5900
+Wire Wire Line
+	4450 6600 4450 6700
+Wire Wire Line
+	3450 6300 3450 6200
+Wire Wire Line
+	3450 6600 3450 6700
+Wire Wire Line
+	3400 6200 3450 6200
+Connection ~ 3450 6200
+Wire Wire Line
+	3450 6200 3450 5900
+Wire Wire Line
+	2450 6600 2450 6700
+Wire Wire Line
+	2450 6700 2450 7300
+Wire Wire Line
+	2400 6200 2450 6200
+Connection ~ 2450 6200
+Wire Wire Line
+	2450 6200 2450 5800
 $EndSCHEMATC

Commit message: Added micro SD slot
Parts:
- added C11: 4.7uF, symbol device:CP
- added C13, C18: 100nF, symbol device:C
- added C7: 10uF, symbol device:CP
- added J10: Micro_SD_Card_Det, Connectors_Card:Hirose_DM3AT-SF-PEJM5, symbol Connector:Micro_SD_Card_Det
- added U3: LT1117-3.3, TO_SOT_Packages_SMD:SOT-223-3_TabPin2, symbol regul:LT1117-2.85
- added U5: 4050, Housings_DIP:SMDIP-14_W7.62mm, symbol Logic_CMOS_4000:4050
- gave numbers to parts that had none: 54
- renumbered C4D02120 to C4D2120
Connections:
- net labels added: +3V3
- wire segments 202 -> 260

Commit message: Added component list and schematic pdf
Parts:
- C1, C10, C12, C13, C14, C15, C18, C2, C4, C6, C8, C9: footprint (none) -> Capacitors_THT:C_Disc_D3.8mm_W2.6mm_P2.50mm
- C11, C16: footprint (none) -> Capacitors_THT:CP_Radial_D5.0mm_P2.00mm
- C17: footprint (none) -> Capacitors_THT:C_Rect_L31.5mm_W20.0mm_P27.50mm_MKS4
- C3: footprint (none) -> Capacitors_THT:CP_Radial_D8.0mm_P5.00mm
- C5: footprint (none) -> Capacitors_THT:CP_Radial_D5.0mm_P2.50mm
- C7: footprint (none) -> Capacitors_THT:CP_Radial_Tantal_D5.0mm_P2.50mm
- CON1: footprint (none) -> Pin_Headers:Pin_Header_Straight_2x03_Pitch2.54mm
- D1, D10, D2, D4, D5, D6, D7, D8, D9: footprint (none) -> Diodes_THT:D_DO-41_SOD81_P10.16mm_Horizontal
- D11: renamed from C4D2120; value D -> C4D2120; footprint (none) -> TO_SOT_Packages_THT:TO-220-2_Vertical
- D3: footprint (none) -> LEDs:LED_D5.0mm
- J1, J11, J5, J6: footprint (none) -> Pin_Headers:Pin_Header_Straight_1x02_Pitch2.54mm
- J12, J7, J8, J9: footprint (none) -> Wire_Pads:SolderWirePad_2x_2mmDrill
- J2, J3, J4: footprint (none) -> Pin_Headers:Pin_Header_Straight_1x03_Pitch2.54mm
- Q1, Q2: footprint (none) -> TO_SOT_Packages_THT:TO-247_TO-3P_Vertical
- R1, R3, R4, R7: footprint (none) -> Resistors_THT:R_Axial_DIN0204_L3.6mm_D1.6mm_P7.62mm_Horizontal
- R10, R2, R5, R6, R8, R9: footprint (none) -> Resistors_THT:R_Axial_DIN0207_L6.3mm_D2.5mm_P10.16mm_Horizontal
- R11: footprint (none) -> Resistors_THT:R_Axial_DIN0411_L9.9mm_D3.6mm_P15.24mm_Horizontal
- SW1: footprint (none) -> Buttons_Switches_THT:SW_PUSH_6mm_h5mm
- U2: value ATMEGA168A-PU -> ATMEGA328P-PU; footprint DIL28 -> Housings_DIP:DIP-28_W7.62mm_LongPads
- U4: footprint Housings_DIP:DIP-8_W7.62mm -> Housings_DIP:DIP-8_W7.62mm_LongPads
- U5: footprint Housings_DIP:SMDIP-14_W7.62mm -> Housings_SOIC:SOIC-16_3.9x9.9mm_Pitch1.27mm
- U5: footprint (none) -> Housings_SOIC:SOIC-16_3.9x9.9mm_Pitch1.27mm
- Y1: footprint (none) -> Crystals:Crystal_HC49-4H_Vertical

Commit message: Generated netlist
Parts:
- J12, J7, J8, J9: footprint Wire_Pads:SolderWirePad_2x_2mmDrill -> HV-WirePad:HV-WirePad
Changed lines of the file:
@@
 F 0 "J7" V 7516 1812 50  0000 R CNN
 F 1 "300V" V 7425 1812 50  0000 R CNN
-F 2 "Wire_Pads:SolderWirePad_2x_2mmDrill" H 7550 2000 50  0001 C CNN
+F 2 "HV-WirePad:HV-WirePad" H 7550 2000 50  0001 C CNN
 F 3 "~" H 7550 2000 50  0001 C CNN
 	1    7550 2000
@@
 F 0 "J8" V 8466 1812 50  0000 R CNN
 F 1 "1200V" V 8375 1812 50  0000 R CNN
-F 2 "Wire_Pads:SolderWirePad_2x_2mmDrill" H 8500 2000 50  0001 C CNN
+F 2 "HV-WirePad:HV-WirePad" H 8500 2000 50  0001 C CNN
 F 3 "~" H 8500 2000 50  0001 C CNN
 	1    8500 2000
@@
 F 0 "J9" V 9316 1812 50  0000 R CNN
 F 1 "Ignitor" V 9225 1812 50  0000 R CNN
-F 2 "Wire_Pads:SolderWirePad_2x_2mmDrill" H 9350 2000 50  0001 C CNN
+F 2 "HV-WirePad:HV-WirePad" H 9350 2000 50  0001 C CNN
 F 3 "~" H 9350 2000 50  0001 C CNN
 	1    9350 2000
@@
 F 0 "J12" V 10516 1812 50  0000 R CNN
 F 1 "Main" V 10425 1812 50  0000 R CNN
-F 2 "Wire_Pads:SolderWirePad_2x_2mmDrill" H 10550 2000 50  0001 C CNN
+F 2 "HV-WirePad:HV-WirePad" H 10550 2000 50  0001 C CNN
 F 3 "~" H 10550 2000 50  0001 C CNN
 	1    10550 2000

Commit message: Layd out all components
Parts:
- removed C7: 10uF, Capacitors_THT:CP_Radial_Tantal_D5.0mm_P2.50mm, symbol device:CP
- D3: footprint LEDs:LED_D5.0mm -> LEDs:LED_D3.0mm
- renumbered C12 to C11, C13 to C12, C14 to C13, C15 to C14, C16 to C15, C17 to C16, C18 to C17, C11 to C7
Connections:
- wire segments 260 -> 256
Changed lines of the file:
@@
 F 0 "D3" V 3038 1233 50  0000 R CNN
 F 1 "LED" V 2947 1233 50  0000 R CNN
-F 2 "LEDs:LED_D5.0mm" H 3000 1350 50  0001 C CNN
+F 2 "LEDs:LED_D3.0mm" H 3000 1350 50  0001 C CNN
 F 3 "~" H 3000 1350 50  0001 C CNN
 	1    3000 1350
@@
 	4500 3450 4500 3950
 $Comp
-L power:GND #PWR017
+L power:GND #PWR018
 U 1 1 5A31FC8C
 P 4500 4050
-F 0 "#PWR017" H 4500 3800 50  0001 C CNN
+F 0 "#PWR018" H 4500 3800 50  0001 C CNN
 F 1 "GND" H 4505 3877 50  0000 C CNN
 F 2 "" H 4500 4050 50  0001 C CNN
@@
 $EndComp
 $Comp
-L power:GND #PWR018
+L power:GND #PWR019
 U 1 1 5A32D1A8
 P 4650 5150
-F 0 "#PWR018" H 4650 4900 50  0001 C CNN
+F 0 "#PWR019" H 4650 4900 50  0001 C CNN
 F 1 "GND" H 4655 4977 50  0000 C CNN
 F 2 "" H 4650 5150 50  0001 C CNN
@@
 	6400 2050 6400 2600
 $Comp
-L device:C C14
+L device:C C13
 U 1 1 5A340DF7
 P 6100 2600
-F 0 "C14" V 5848 2600 50  0000 C CNN
+F 0 "C13" V 5848 2600 50  0000 C CNN
 F 1 "100nF" V 5939 2600 50  0000 C CNN
 F 2 "Capacitors_THT:C_Disc_D3.8mm_W2.6mm_P2.50mm" H 6138 2450 50  0001 C CNN
@@
 18V
 $Comp
-L device:CP C16
+L device:CP C15
 U 1 1 5A369449
 P 6900 5000
-F 0 "C16" H 7018 5046 50  0000 L CNN
+F 0 "C15" H 7018 5046 50  0000 L CNN
 F 1 "4.7uF" H 7018 4955 50  0000 L CNN
 F 2 "Capacitors_THT:CP_Radial_D5.0mm_P2.00mm" H 6938 4850 50  0001 C CNN
@@
 $EndComp
 $Comp
-L device:C C15
+L device:C C14
 U 1 1 5A3696D9
 P 6350 5000
-F 0 "C15" H 6465 5046 50  0000 L CNN
+F 0 "C14" H 6465 5046 50  0000 L CNN
 F 1 "100nF" H 6465 4955 50  0000 L CNN
 F 2 "Capacitors_THT:C_Disc_D3.8mm_W2.6mm_P2.50mm" H 6388 4850 50  0001 C CNN
@@
 	7550 2300 7550 2200
 $Comp
-L device:C C17
+L device:C C16
 U 1 1 5A310386
 P 7700 2800
-F 0 "C17" V 7448 2800 50  0000 C CNN
+F 0 "C16" V 7448 2800 50  0000 C CNN
 F 1 "5uF" V 7539 2800 50  0000 C CNN
 F 2 "Capacitors_THT:C_Rect_L31.5mm_W20.0mm_P27.50mm_MKS4" H 7738 2650 50  0001 C CNN
@@
 	4400 6700 4450 6700
 $Comp
-L power:+5V #PWR020
+L power:+5V #PWR021
 U 1 1 5A4955E9
 P 4850 6600
-F 0 "#PWR020" H 4850 6450 50  0001 C CNN
+F 0 "#PWR021" H 4850 6450 50  0001 C CNN
 F 1 "+5V" H 4865 6773 50  0000 C CNN
 F 2 "" H 4850 6600 50  0001 C CNN
@@
 $EndComp
 $Comp
-L device:C C12
+L device:C C11
 U 1 1 5A49A31A
 P 5250 6200
-F 0 "C12" V 4998 6200 50  0000 C CNN
+F 0 "C11" V 4998 6200 50  0000 C CNN
 F 1 "10nF" V 5089 6200 50  0000 C CNN
 F 2 "Capacitors_THT:C_Disc_D3.8mm_W2.6mm_P2.50mm" H 5288 6050 50  0001 C CNN
@@
 $EndComp
 $Comp
-L power:+5V #PWR019
+L power:+5V #PWR020
 U 1 1 5A5BFD8B
 P 4750 7300
-F 0 "#PWR019" H 4750 7150 50  0001 C CNN
+F 0 "#PWR020" H 4750 7150 50  0001 C CNN
 F 1 "+5V" H 4765 7473 50  0000 C CNN
 F 2 "" H 4750 7300 50  0001 C CNN
@@
 L regul:LT1117-2.85 U3
 U 1 1 5A3261F2
-P 4150 800
-F 0 "U3" H 4150 1042 50  0000 C CNN
-F 1 "LT1117-3.3" H 4150 951 50  0000 C CNN
-F 2 "TO_SOT_Packages_SMD:SOT-223-3_TabPin2" H 4150 800 50  0001 C CNN
-F 3 "http://cds.linear.com/docs/en/datasheet/1117fd.pdf" H 4150 800 50  0001 C CNN
-	1    4150 800
-	1    0    0    -1
-$EndComp
-$Comp
-L power:+3V3 #PWR021
+P 3650 800
+F 0 "U3" H 3650 1042 50  0000 C CNN
+F 1 "LT1117-3.3" H 3650 951 50  0000 C CNN
+F 2 "TO_SOT_Packages_SMD:SOT-223-3_TabPin2" H 3650 800 50  0001 C CNN
+F 3 "http://cds.linear.com/docs/en/datasheet/1117fd.pdf" H 3650 800 50  0001 C CNN
+	1    3650 800
+	1    0    0    -1
+$EndComp
+$Comp
+L power:+3V3 #PWR017
 U 1 1 5A368866
-P 5050 800
-F 0 "#PWR021" H 5050 650 50  0001 C CNN
-F 1 "+3V3" H 5065 973 50  0000 C CNN
-F 2 "" H 5050 800 50  0001 C CNN
-F 3 "" H 5050 800 50  0001 C CNN
-	1    5050 800
-	1    0    0    -1
-$EndComp
-$Comp
-L device:CP C7
-U 1 1 5A3690BA
-P 3550 1150
-F 0 "C7" H 3668 1196 50  0000 L CNN
-F 1 "10uF" H 3668 1105 50  0000 L CNN
-F 2 "Capacitors_THT:CP_Radial_Tantal_D5.0mm_P2.50mm" H 3588 1000 50  0001 C CNN
-F 3 "" H 3550 1150 50  0001 C CNN
-	1    3550 1150
-	1    0    0    -1
-$EndComp
-Wire Wire Line
-	3000 800  3550 800
-Wire Wire Line
-	4450 800  4750 800
-Wire Wire Line
-	4750 800  4750 950
-Connection ~ 4750 800
-Wire Wire Line
-	4750 800  5050 800
-Wire Wire Line
-	3000 1500 3550 1500
-Wire Wire Line
-	4750 1500 4750 1250
-Wire Wire Line
-	4150 1100 4150 1500
-Connection ~ 4150 1500
-Wire Wire Line
-	4150 1500 4750 1500
+P 4450 800
+F 0 "#PWR017" H 4450 650 50  0001 C CNN
+F 1 "+3V3" H 4465 973 50  0000 C CNN
+F 2 "" H 4450 800 50  0001 C CNN
+F 3 "" H 4450 800 50  0001 C CNN
+	1    4450 800
+	1    0    0    -1
+$EndComp
+Wire Wire Line
+	3950 800  4150 800
+Wire Wire Line
+	4150 800  4150 950
+Connection ~ 4150 800
+Wire Wire Line
+	4150 800  4450 800
+Wire Wire Line
+	4150 1500 4150 1250
+Wire Wire Line
+	3650 1100 3650 1500
+Connection ~ 3650 1500
+Wire Wire Line
+	3650 1500 4150 1500
 Wire Wire Line
 	7900 5550 7900 4050
@@
 	9750 4050 9750 3150
 Connection ~ 3000 1500
-Wire Wire Line
-	3550 1300 3550 1500
-Connection ~ 3550 1500
-Wire Wire Line
-	3550 1500 4150 1500
-Wire Wire Line
-	3550 1000 3550 800
-Connection ~ 3550 800
-Wire Wire Line
-	3550 800  3850 800
-$Comp
-L device:CP C11
+$Comp
+L device:CP C7
 U 1 1 5A4B9E54
-P 4750 1100
-F 0 "C11" H 4868 1146 50  0000 L CNN
-F 1 "4.7uF" H 4868 1055 50  0000 L CNN
-F 2 "Capacitors_THT:CP_Radial_D5.0mm_P2.00mm" H 4788 950 50  0001 C CNN
-F 3 "" H 4750 1100 50  0001 C CNN
-	1    4750 1100
+P 4150 1100
+F 0 "C7" H 4268 1146 50  0000 L CNN
+F 1 "4.7uF" H 4268 1055 50  0000 L CNN
+F 2 "Capacitors_THT:CP_Radial_D5.0mm_P2.00mm" H 4188 950 50  0001 C CNN
+F 3 "" H 4150 1100 50  0001 C CNN
+	1    4150 1100
 	1    0    0    -1
 $EndComp
@@
 	5400 950  5500 950
 $Comp
-L device:C C13
+L device:C C12
 U 1 1 5A547015
 P 5500 1200
-F 0 "C13" H 5615 1246 50  0000 L CNN
+F 0 "C12" H 5615 1246 50  0000 L CNN
 F 1 "100nF" H 5615 1155 50  0000 L CNN
 F 2 "Capacitors_THT:C_Disc_D3.8mm_W2.6mm_P2.50mm" H 5538 1050 50  0001 C CNN
@@
 $EndComp
 $Comp
-L device:C C18
+L device:C C17
 U 1 1 5AAE419A
 P 9300 4500
-F 0 "C18" H 9415 4546 50  0000 L CNN
+F 0 "C17" H 9415 4546 50  0000 L CNN
 F 1 "100nF" H 9415 4455 50  0000 L CNN
 F 2 "Capacitors_THT:C_Disc_D3.8mm_W2.6mm_P2.50mm" H 9338 4350 50  0001 C CNN
@@
 Wire Wire Line
 	9450 4500 9550 4500
+Wire Wire Line
+	3000 800  3350 800
+Wire Wire Line
+	3000 1500 3650 1500
 $EndSCHEMATC
