File: Elephant-3/Elephant-3.sch (KiCad schematic (older format))
At the start: 61 parts, among them CON1 AVR-ISP-6, J1 7-25V, J10 Micro_SD_Card_Det, J11 IgnCap, J12 Main, J2 ADC2, J3 ADC1, J4 ADC0, J5 Switch, J6 18V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

Commit message: Routed through hole pcb
Connections:
- net labels removed: +18V
Changed lines of the file:
@@
 Sheet 1 1
 Title "Elephant-3 Control Board"
-Date "2017-12-13"
+Date "2017-12-14"
 Rev "1"
 Comp ""
@@
 $EndComp
 Text GLabel 7250 4850 2    60   Input ~ 0
-+18V
+18V
 $Comp
 L device:C C1

Commit message: Labeled stuff on PCB
Parts:
- CON1: value AVR-ISP-6 -> ISP
- J10: value Micro_SD_Card_Det -> Micro_SD_Card
- U1: value LM7805_TO220 -> LM7805
- U2: value ATMEGA328P-PU -> ATMEGA328
- U3: value LT1117-3.3 -> LT1117
Changed lines of the file:
@@
 P 4750 2200
 F 0 "CON1" V 4383 2250 50  0000 C CNN
-F 1 "AVR-ISP-6" V 4474 2250 50  0000 C CNN
+F 1 "ISP" V 4474 2250 50  0000 C CNN
 F 2 "Pin_Headers:Pin_Header_Straight_2x03_Pitch2.54mm" V 4500 2250 50  0001 C CNN
 F 3 "" H 3475 1650 50  0001 C CNN
@@
 P 2400 3950
 F 0 "U2" H 2450 5317 50  0000 C CNN
-F 1 "ATMEGA328P-PU" H 2450 5226 50  0000 C CNN
+F 1 "ATMEGA328" H 2450 5226 50  0000 C CNN
 F 2 "Housings_DIP:DIP-28_W7.62mm_LongPads" H 2400 3950 50  0001 C CIN
 F 3 "http://www.atmel.com/images/atmel-8271-8-bit-avr-microcontroller-atmega48a-48pa-88a-88pa-168a-168pa-328-328p_datasheet.pdf" H 2400 3950 50  0001 C CNN
@@
 P 1850 800
 F 0 "U1" H 1850 1042 50  0000 C CNN
-F 1 "LM7805_TO220" H 1850 951 50  0000 C CNN
+F 1 "LM7805" H 1850 951 50  0000 C CNN
 F 2 "TO_SOT_Packages_THT:TO-220-3_Vertical" H 1850 1025 50  0001 C CIN
 F 3 "http://www.fairchildsemi.com/ds/LM/LM7805.pdf" H 1850 750 50  0001 C CNN
@@
 P 3650 800
 F 0 "U3" H 3650 1042 50  0000 C CNN
-F 1 "LT1117-3.3" H 3650 951 50  0000 C CNN
+F 1 "LT1117" H 3650 951 50  0000 C CNN
 F 2 "TO_SOT_Packages_SMD:SOT-223-3_TabPin2" H 3650 800 50  0001 C CNN
 F 3 "http://cds.linear.com/docs/en/datasheet/1117fd.pdf" H 3650 800 50  0001 C CNN
@@
 P 10000 5500
 F 0 "J10" H 9950 6317 50  0000 C CNN
-F 1 "Micro_SD_Card_Det" H 9950 6226 50  0000 C CNN
+F 1 "Micro_SD_Card" H 9950 6226 50  0000 C CNN
 F 2 "Connectors_Card:Hirose_DM3AT-SF-PEJM5" H 12050 6200 50  0001 C CNN
 F 3 "https://www.hirose.com/product/en/download_file/key_name/DM3/category/Catalog/doc_file_id/49662/?file_category_id=4&item_id=195&is_series=1" H 10000 5600 50  0001 C CNN

Commit message: Added project files for smd version and replaced some component to generic
Parts:
- D11: value C4D2120 -> D
Changed lines of the file:
@@
 P 7850 2400
 F 0 "D11" V 7896 2321 50  0000 R CNN
-F 1 "C4D2120" V 7805 2321 50  0000 R CNN
+F 1 "D" V 7805 2321 50  0000 R CNN
 F 2 "TO_SOT_Packages_THT:TO-220-2_Vertical" H 7850 2400 50  0001 C CNN
 F 3 "" H 7850 2400 50  0001 C CNN
