File: Elephant-3/Elephant-3.kicad_pcb (KiCad board)
At the start: 2 copper layers, 90.2 x 58.4 mm, 61 parts, among them CON1 AVR-ISP-6, J1 7-25V, J10 Micro_SD_Card_Det, J11 IgnCap, J12 Main, J2 ADC2, J3 ADC1, J4 ADC0, J5 Switch, J6 18V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

Commit message: Routed through hole pcb
Parts:
- moved C17 25.8 mm to (115.6, 107.3), turned to 180 degrees
- moved C12 11.5 mm to (126.9, 105.4)
- moved SW1 8.15 mm to (132.8, 125.0), turned to 180 degrees
- moved C7 8.05 mm to (127.3, 99.2), turned to 0 degrees
- moved U3 7.62 mm to (120.9, 103.5)
- moved D1 5.08 mm to (160.7, 125.1)
- moved D2 5.08 mm to (155.6, 114.9)
- moved R5 2.79 mm to (131.4, 95.0)
- moved D3 2.71 mm to (151.9, 95.1)
- moved J1 2.54 mm to (115.6, 71.1), turned to 90 degrees
- moved J6 2.54 mm to (124.5, 71.1), turned to 90 degrees
- moved R2 1.80 mm to (156.7, 105.4)
- moved C10 1.55 mm to (138.2, 120.9), turned to 90 degrees
- moved U5 1.55 mm to (129.3, 111.5), turned to 0 degrees
- moved D8 0.64 mm to (142.2, 81.9)
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Connections:
- C14 pad 1: +18V -> 18V
- C15 pad 1: +18V -> 18V
- U4 pad 6: +18V -> 18V
Routing:
- net +5V: track 0.00 -> 209.9 mm, vias 0 -> 2
- net Net-(C13-Pad2): track 0.00 -> 108.2 mm
- net 300V: track 0.00 -> 69.9 mm
- net IgnCap: track 0.00 -> 67.4 mm, vias 0 -> 2
- net Net-(CON1-Pad1): track 0.00 -> 67.3 mm
- net Net-(Q2-Pad1): track 0.00 -> 62.6 mm, vias 0 -> 2
- net Net-(U2-Pad13): track 0.00 -> 60.5 mm, vias 0 -> 4
- net Net-(Q1-Pad1): track 0.00 -> 58.8 mm, vias 0 -> 2
- net Net-(U2-Pad11): track 0.00 -> 53.8 mm, vias 0 -> 4
- net Net-(CON1-Pad3): track 0.00 -> 53.1 mm
- net 18V: track 0.00 -> 51.1 mm
- net Net-(CON1-Pad4): track 0.00 -> 43.8 mm
- net Net-(J5-Pad1): track 0.00 -> 41.9 mm, vias 0 -> 1
- net Net-(C11-Pad1): track 0.00 -> 37.3 mm, vias 0 -> 2
- net Net-(C4-Pad1): track 0.00 -> 37.0 mm
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Other:
- net class 1200V: trace_width 2 -> 3
- net class 1200V-excp: trace_width 2 -> 3
- net class 300V: trace_width 0.25 -> 2
- net class 300V-signal added: clearance 1, trace_width 0.5, via_dia 0.8, via_drill 0.4
- net class Power added: clearance 0.2, trace_width 0.5, via_dia 0.8, via_drill 0.4
