File: Elephant-3/Elephant-3.kicad_pcb (KiCad board)
At the start: 2 copper layers, 90.2 x 58.4 mm, 61 parts, among them CON1 ISP, J1 7-25V, J10 Micro_SD_Card, J11 IgnCap, J12 Main, J2 ADC2, J3 ADC1, J4 ADC0, J5 Switch, J6 18V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

Commit message: Added name/version on to pcb
Other:
- board text added: "Designed by Corwin Hansen UW APL Ver. 1.0"
Changed lines of the file:
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@@
   (general
     (thickness 1.6)
-    (drawings 19)
+    (drawings 20)
     (tracks 485)
     (zones 0)
@@
     )
   )
+  (gr_text "Designed by Corwin Hansen   UW APL  Ver. 1.0\n" (at 169.164 86.106) (layer B.SilkS)
+    (effects (font (size 1 1) (thickness 0.25)) (justify mirror))
+  )
   (gr_text - (at 197.104 126.365 180) (layer F.SilkS)
