File: Elephant-3_smd/Elephant-3.sch (KiCad schematic (older format))
At the start: 61 parts, among them CON1 ISP, J1 7-25V, J10 Micro_SD_Card, J11 IgnCap, J12 Main, J2 ADC2, J3 ADC1, J4 ADC0, J5 Switch, J6 18V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

Commit message: Added project files for smd version and replaced some component to generic
Parts:
- removed U2: ATMEGA328, Housings_DIP:DIP-28_W7.62mm_LongPads, symbol atmel:ATMEGA168A-PU
- added U2: ATMEGA328, Housings_QFP:TQFP-32_7x7mm_Pitch0.8mm, symbol atmel:ATMEGA168A-AU
- D11: value C4D2120 -> D
Connections:
- wire segments 256 -> 259
Changed lines of the file:
@@
-	1    0    0    -1
-$EndComp
-$Comp
-L atmel:ATMEGA168A-PU U2
-U 1 1 5A2FD10A
-P 2400 3950
-F 0 "U2" H 2450 5317 50  0000 C CNN
-F 1 "ATMEGA328" H 2450 5226 50  0000 C CNN
-F 2 "Housings_DIP:DIP-28_W7.62mm_LongPads" H 2400 3950 50  0001 C CIN
-F 3 "http://www.atmel.com/images/atmel-8271-8-bit-avr-microcontroller-atmega48a-48pa-88a-88pa-168a-168pa-328-328p_datasheet.pdf" H 2400 3950 50  0001 C CNN
-	1    2400 3950
 	1    0    0    -1
 $EndComp
@@
 P 7850 2400
 F 0 "D11" V 7896 2321 50  0000 R CNN
-F 1 "C4D2120" V 7805 2321 50  0000 R CNN
+F 1 "D" V 7805 2321 50  0000 R CNN
 F 2 "TO_SOT_Packages_THT:TO-220-2_Vertical" H 7850 2400 50  0001 C CNN
 F 3 "" H 7850 2400 50  0001 C CNN
@@
 Wire Wire Line
 	3000 1500 3650 1500
+$Comp
+L atmel:ATMEGA168A-AU U2
+U 1 1 5A46F45C
+P 2400 3950
+F 0 "U2" H 2450 5317 50  0000 C CNN
+F 1 "ATMEGA328" H 2450 5226 50  0000 C CNN
+F 2 "Housings_QFP:TQFP-32_7x7mm_Pitch0.8mm" H 2400 3950 50  0001 C CIN
+F 3 "http://www.atmel.com/images/atmel-8271-8-bit-avr-microcontroller-atmega48a-48pa-88a-88pa-168a-168pa-328-328p_datasheet.pdf" H 2400 3950 50  0001 C CNN
+	1    2400 3950
+	1    0    0    -1
+$EndComp
+Wire Wire Line
+	1500 2950 1500 2850
+Connection ~ 1500 2850
+Wire Wire Line
+	1500 4950 950  4950
+Wire Wire Line
+	950  4950 950  5050
+Connection ~ 950  5050
 $EndSCHEMATC

Commit message: Got component list
Parts:
- CON1: footprint Pin_Headers:Pin_Header_Straight_2x03_Pitch2.54mm -> Pin_Headers:Pin_Header_Straight_2x03_Pitch2.54mm_SMD
- SW1: footprint Buttons_Switches_THT:SW_PUSH_6mm_h5mm -> Buttons_Switches_SMD:SW_SPST_PTS645
- U1: value LM7805 -> 7805; footprint TO_SOT_Packages_THT:TO-220-3_Vertical -> TO_SOT_Packages_SMD:TO-252-3_TabPin2
- Y1: footprint Crystals:Crystal_HC49-4H_Vertical -> Crystals:Crystal_SMD_SeikoEpson_FA238-4pin_3.2x2.5mm_HandSoldering
Changed lines of the file:
@@
 F 0 "CON1" V 4383 2250 50  0000 C CNN
 F 1 "ISP" V 4474 2250 50  0000 C CNN
-F 2 "Pin_Headers:Pin_Header_Straight_2x03_Pitch2.54mm" V 4500 2250 50  0001 C CNN
+F 2 "Pin_Headers:Pin_Header_Straight_2x03_Pitch2.54mm_SMD" V 4500 2250 50  0001 C CNN
 F 3 "" H 3475 1650 50  0001 C CNN
 	1    4750 2200
@@
 P 1850 800
 F 0 "U1" H 1850 1042 50  0000 C CNN
-F 1 "LM7805" H 1850 951 50  0000 C CNN
-F 2 "TO_SOT_Packages_THT:TO-220-3_Vertical" H 1850 1025 50  0001 C CIN
+F 1 "7805" H 1850 951 50  0000 C CNN
+F 2 "TO_SOT_Packages_SMD:TO-252-3_TabPin2" H 1850 1025 50  0001 C CIN
 F 3 "http://www.fairchildsemi.com/ds/LM/LM7805.pdf" H 1850 750 50  0001 C CNN
 	1    1850 800
@@
 F 0 "Y1" V 3854 3731 50  0000 L CNN
 F 1 "16MHz" V 3945 3731 50  0000 L CNN
-F 2 "Crystals:Crystal_HC49-4H_Vertical" H 3900 3600 50  0001 C CNN
+F 2 "Crystals:Crystal_SMD_SeikoEpson_FA238-4pin_3.2x2.5mm_HandSoldering" H 3900 3600 50  0001 C CNN
 F 3 "" H 3900 3600 50  0001 C CNN
 	1    3900 3600
@@
 F 0 "SW1" H 6100 2317 50  0000 C CNN
 F 1 "Reset" H 6100 2226 50  0000 C CNN
-F 2 "Buttons_Switches_THT:SW_PUSH_6mm_h5mm" H 6100 2050 50  0001 C CNN
+F 2 "Buttons_Switches_SMD:SW_SPST_PTS645" H 6100 2050 50  0001 C CNN
 F 3 "" H 6100 2050 50  0001 C CNN
 	1    6100 2050

Commit message: Generated netlist for smd
Parts:
- C1, C12, C13, C14, C17, C2: footprint Capacitors_THT:C_Disc_D3.8mm_W2.6mm_P2.50mm -> Capacitors_SMD:C_0603
- C10, C11, C4, C6, C8, C9: footprint Capacitors_THT:C_Disc_D3.8mm_W2.6mm_P2.50mm -> Capacitors_SMD:C_0402
- C3: footprint Capacitors_THT:CP_Radial_D8.0mm_P5.00mm -> Capacitors_SMD:CP_Elec_6.3x5.3
- C5: footprint Capacitors_THT:CP_Radial_D5.0mm_P2.50mm -> Capacitors_SMD:CP_Elec_5x5.3
- C7: footprint Capacitors_THT:CP_Radial_D5.0mm_P2.00mm -> Capacitors_SMD:CP_Elec_4x5.3
- D1, D10, D2, D4, D5, D6, D7, D8, D9: footprint Diodes_THT:D_DO-41_SOD81_P10.16mm_Horizontal -> Diodes_SMD:D_SMA
- D3: footprint LEDs:LED_D3.0mm -> LEDs:LED_0805
- R1, R3, R4, R7: footprint Resistors_THT:R_Axial_DIN0204_L3.6mm_D1.6mm_P7.62mm_Horizontal -> Resistors_SMD:R_0402
- R10, R5, R6, R8, R9: footprint Resistors_THT:R_Axial_DIN0207_L6.3mm_D2.5mm_P10.16mm_Horizontal -> Resistors_SMD:R_1206
- R11: footprint Resistors_THT:R_Axial_DIN0411_L9.9mm_D3.6mm_P15.24mm_Horizontal -> Resistors_SMD:R_0805
- R2: footprint Resistors_THT:R_Axial_DIN0207_L6.3mm_D2.5mm_P10.16mm_Horizontal -> Resistors_SMD:R_0805
Changed lines of the file:
@@
 F 0 "C1" H 1115 2396 50  0000 L CNN
 F 1 "100nF" H 1115 2305 50  0000 L CNN
-F 2 "Capacitors_THT:C_Disc_D3.8mm_W2.6mm_P2.50mm" H 1038 2200 50  0001 C CNN
+F 2 "Capacitors_SMD:C_0603" H 1038 2200 50  0001 C CNN
 F 3 "" H 1000 2350 50  0001 C CNN
 	1    1000 2350
@@
 F 0 "C5" H 2618 1196 50  0000 L CNN
 F 1 "10uF" H 2618 1105 50  0000 L CNN
-F 2 "Capacitors_THT:CP_Radial_D5.0mm_P2.50mm" H 2538 1000 50  0001 C CNN
+F 2 "Capacitors_SMD:CP_Elec_5x5.3" H 2538 1000 50  0001 C CNN
 F 3 "" H 2500 1150 50  0001 C CNN
 	1    2500 1150
@@
 F 0 "C3" H 1368 1196 50  0000 L CNN
 F 1 "100uF" H 1368 1105 50  0000 L CNN
-F 2 "Capacitors_THT:CP_Radial_D8.0mm_P5.00mm" H 1288 1000 50  0001 C CNN
+F 2 "Capacitors_SMD:CP_Elec_6.3x5.3" H 1288 1000 50  0001 C CNN
 F 3 "" H 1250 1150 50  0001 C CNN
 	1    1250 1150
@@
 F 0 "D3" V 3038 1233 50  0000 R CNN
 F 1 "LED" V 2947 1233 50  0000 R CNN
-F 2 "LEDs:LED_D3.0mm" H 3000 1350 50  0001 C CNN
+F 2 "LEDs:LED_0805" H 3000 1350 50  0001 C CNN
 F 3 "~" H 3000 1350 50  0001 C CNN
 	1    3000 1350
@@
 F 0 "R2" H 3070 1046 50  0000 L CNN
 F 1 "150" H 3070 955 50  0000 L CNN
-F 2 "Resistors_THT:R_Axial_DIN0207_L6.3mm_D2.5mm_P10.16mm_Horizontal" V 2930 1000 50  0001 C CNN
+F 2 "Resistors_SMD:R_0805" V 2930 1000 50  0001 C CNN
 F 3 "" H 3000 1000 50  0001 C CNN
 	1    3000 1000
@@
 F 0 "C9" V 4098 3450 50  0000 C CNN
 F 1 "22pF" V 4189 3450 50  0000 C CNN
-F 2 "Capacitors_THT:C_Disc_D3.8mm_W2.6mm_P2.50mm" H 4388 3300 50  0001 C CNN
+F 2 "Capacitors_SMD:C_0402" H 4388 3300 50  0001 C CNN
 F 3 "" H 4350 3450 50  0001 C CNN
 	1    4350 3450
@@
 F 0 "C10" V 4098 3950 50  0000 C CNN
 F 1 "22pF" V 4189 3950 50  0000 C CNN
-F 2 "Capacitors_THT:C_Disc_D3.8mm_W2.6mm_P2.50mm" H 4388 3800 50  0001 C CNN
+F 2 "Capacitors_SMD:C_0402" H 4388 3800 50  0001 C CNN
 F 3 "" H 4350 3950 50  0001 C CNN
 	1    4350 3950
@@
 F 0 "R5" H 4580 4754 50  0000 R CNN
 F 1 "10k" H 4580 4845 50  0000 R CNN
-F 2 "Resistors_THT:R_Axial_DIN0207_L6.3mm_D2.5mm_P10.16mm_Horizontal" V 4580 4800 50  0001 C CNN
+F 2 "Resistors_SMD:R_1206" V 4580 4800 50  0001 C CNN
 F 3 "" H 4650 4800 50  0001 C CNN
 	1    4650 4800
@@
 F 0 "R6" H 5320 4046 50  0000 L CNN
 F 1 "10k" H 5320 3955 50  0000 L CNN
-F 2 "Resistors_THT:R_Axial_DIN0207_L6.3mm_D2.5mm_P10.16mm_Horizontal" V 5180 4000 50  0001 C CNN
+F 2 "Resistors_SMD:R_1206" V 5180 4000 50  0001 C CNN
 F 3 "" H 5250 4000 50  0001 C CNN
 	1    5250 4000
@@
 F 0 "C13" V 5848 2600 50  0000 C CNN
 F 1 "100nF" V 5939 2600 50  0000 C CNN
-F 2 "Capacitors_THT:C_Disc_D3.8mm_W2.6mm_P2.50mm" H 6138 2450 50  0001 C CNN
+F 2 "Capacitors_SMD:C_0603" H 6138 2450 50  0001 C CNN
 F 3 "" H 6100 2600 50  0001 C CNN
 	1    6100 2600
@@
 F 0 "D8" V 4954 4079 50  0000 L CNN
 F 1 "D" V 5045 4079 50  0000 L CNN
-F 2 "Diodes_THT:D_DO-41_SOD81_P10.16mm_Horizontal" H 5000 4000 50  0001 C CNN
+F 2 "Diodes_SMD:D_SMA" H 5000 4000 50  0001 C CNN
 F 3 "" H 5000 4000 50  0001 C CNN
 	1    5000 4000
@@
 F 0 "C2" H 1115 3346 50  0000 L CNN
 F 1 "100nF" H 1115 3255 50  0000 L CNN
-F 2 "Capacitors_THT:C_Disc_D3.8mm_W2.6mm_P2.50mm" H 1038 3150 50  0001 C CNN
+F 2 "Capacitors_SMD:C_0603" H 1038 3150 50  0001 C CNN
 F 3 "" H 1000 3300 50  0001 C CNN
 	1    1000 3300
@@
 F 0 "C14" H 6465 5046 50  0000 L CNN
 F 1 "100nF" H 6465 4955 50  0000 L CNN
-F 2 "Capacitors_THT:C_Disc_D3.8mm_W2.6mm_P2.50mm" H 6388 4850 50  0001 C CNN
+F 2 "Capacitors_SMD:C_0603" H 6388 4850 50  0001 C CNN
 F 3 "" H 6350 5000 50  0001 C CNN
 	1    6350 5000
@@
 F 0 "D4" V 3204 6779 50  0000 L CNN
 F 1 "D_Schottky" V 3295 6779 50  0000 L CNN
-F 2 "Diodes_THT:D_DO-41_SOD81_P10.16mm_Horizontal" H 3250 6700 50  0001 C CNN
+F 2 "Diodes_SMD:D_SMA" H 3250 6700 50  0001 C CNN
 F 3 "" H 3250 6700 50  0001 C CNN
 	1    3250 6700
@@
 F 0 "R8" H 8820 3446 50  0000 L CNN
 F 1 "340k" H 8820 3355 50  0000 L CNN
-F 2 "Resistors_THT:R_Axial_DIN0207_L6.3mm_D2.5mm_P10.16mm_Horizontal" V 8680 3400 50  0001 C CNN
+F 2 "Resistors_SMD:R_1206" V 8680 3400 50  0001 C CNN
 F 3 "" H 8750 3400 50  0001 C CNN
 	1    8750 3400
@@
 F 0 "R10" H 10020 3446 50  0000 L CNN
 F 1 "340k" H 10020 3355 50  0000 L CNN
-F 2 "Resistors_THT:R_Axial_DIN0207_L6.3mm_D2.5mm_P10.16mm_Horizontal" V 9880 3400 50  0001 C CNN
+F 2 "Resistors_SMD:R_1206" V 9880 3400 50  0001 C CNN
 F 3 "" H 9950 3400 50  0001 C CNN
 	1    9950 3400
@@
 F 0 "D5" V 3604 6779 50  0000 L CNN
 F 1 "D_Schottky" V 3695 6779 50  0000 L CNN
-F 2 "Diodes_THT:D_DO-41_SOD81_P10.16mm_Horizontal" H 3650 6700 50  0001 C CNN
+F 2 "Diodes_SMD:D_SMA" H 3650 6700 50  0001 C CNN
 F 3 "" H 3650 6700 50  0001 C CNN
 	1    3650 6700
@@
 F 0 "R3" H 3520 6496 50  0000 L CNN
 F 1 "680" H 3520 6405 50  0000 L CNN
-F 2 "Resistors_THT:R_Axial_DIN0204_L3.6mm_D1.6mm_P7.62mm_Horizontal" V 3380 6450 50  0001 C CNN
+F 2 "Resistors_SMD:R_0402" V 3380 6450 50  0001 C CNN
 F 3 "" H 3450 6450 50  0001 C CNN
 	1    3450 6450
@@
 F 0 "C6" V 2998 6200 50  0000 C CNN
 F 1 "10nF" V 3089 6200 50  0000 C CNN
-F 2 "Capacitors_THT:C_Disc_D3.8mm_W2.6mm_P2.50mm" H 3288 6050 50  0001 C CNN
+F 2 "Capacitors_SMD:C_0402" H 3288 6050 50  0001 C CNN
 F 3 "" H 3250 6200 50  0001 C CNN
 	1    3250 6200
@@
 F 0 "D6" V 4204 6779 50  0000 L CNN
 F 1 "D_Schottky" V 4295 6779 50  0000 L CNN
-F 2 "Diodes_THT:D_DO-41_SOD81_P10.16mm_Horizontal" H 4250 6700 50  0001 C CNN
+F 2 "Diodes_SMD:D_SMA" H 4250 6700 50  0001 C CNN
 F 3 "" H 4250 6700 50  0001 C CNN
 	1    4250 6700
@@
 F 0 "D7" V 4604 6779 50  0000 L CNN
 F 1 "D_Schottky" V 4695 6779 50  0000 L CNN
-F 2 "Diodes_THT:D_DO-41_SOD81_P10.16mm_Horizontal" H 4650 6700 50  0001 C CNN
+F 2 "Diodes_SMD:D_SMA" H 4650 6700 50  0001 C CNN
 F 3 "" H 4650 6700 50  0001 C CNN
 	1    4650 6700
@@
 F 0 "R4" H 4520 6496 50  0000 L CNN
 F 1 "680" H 4520 6405 50  0000 L CNN
-F 2 "Resistors_THT:R_Axial_DIN0204_L3.6mm_D1.6mm_P7.62mm_Horizontal" V 4380 6450 50  0001 C CNN
+F 2 "Resistors_SMD:R_0402" V 4380 6450 50  0001 C CNN
 F 3 "" H 4450 6450 50  0001 C CNN
 	1    4450 6450
@@
 F 0 "C8" V 3998 6200 50  0000 C CNN
 F 1 "10nF" V 4089 6200 50  0000 C CNN
-F 2 "Capacitors_THT:C_Disc_D3.8mm_W2.6mm_P2.50mm" H 4288 6050 50  0001 C CNN
+F 2 "Capacitors_SMD:C_0402" H 4288 6050 50  0001 C CNN
 F 3 "" H 4250 6200 50  0001 C CNN
 	1    4250 6200
@@
 F 0 "D9" V 5204 6779 50  0000 L CNN
 F 1 "D_Schottky" V 5295 6779 50  0000 L CNN
-F 2 "Diodes_THT:D_DO-41_SOD81_P10.16mm_Horizontal" H 5250 6700 50  0001 C CNN
+F 2 "Diodes_SMD:D_SMA" H 5250 6700 50  0001 C CNN
 F 3 "" H 5250 6700 50  0001 C CNN
 	1    5250 6700
@@
 F 0 "D10" V 5604 6779 50  0000 L CNN
 F 1 "D_Schottky" V 5695 6779 50  0000 L CNN
-F 2 "Diodes_THT:D_DO-41_SOD81_P10.16mm_Horizontal" H 5650 6700 50  0001 C CNN
+F 2 "Diodes_SMD:D_SMA" H 5650 6700 50  0001 C CNN
 F 3 "" H 5650 6700 50  0001 C CNN
 	1    5650 6700
@@
 F 0 "R7" H 5520 6496 50  0000 L CNN
 F 1 "680" H 5520 6405 50  0000 L CNN
-F 2 "Resistors_THT:R_Axial_DIN0204_L3.6mm_D1.6mm_P7.62mm_Horizontal" V 5380 6450 50  0001 C CNN
+F 2 "Resistors_SMD:R_0402" V 5380 6450 50  0001 C CNN
 F 3 "" H 5450 6450 50  0001 C CNN
 	1    5450 6450
@@
 F 0 "C11" V 4998 6200 50  0000 C CNN
 F 1 "10nF" V 5089 6200 50  0000 C CNN
-F 2 "Capacitors_THT:C_Disc_D3.8mm_W2.6mm_P2.50mm" H 5288 6050 50  0001 C CNN
+F 2 "Capacitors_SMD:C_0402" H 5288 6050 50  0001 C CNN
 F 3 "" H 5250 6200 50  0001 C CNN
 	1    5250 6200
@@
 F 0 "R9" V 9643 1150 50  0000 C CNN
 F 1 "10k" V 9734 1150 50  0000 C CNN
-F 2 "Resistors_THT:R_Axial_DIN0207_L6.3mm_D2.5mm_P10.16mm_Horizontal" V 9780 1150 50  0001 C CNN
+F 2 "Resistors_SMD:R_1206" V 9780 1150 50  0001 C CNN
 F 3 "" H 9850 1150 50  0001 C CNN
 	1    9850 1150
@@
 F 0 "R11" V 10293 1150 50  0000 C CNN
 F 1 "680k" V 10384 1150 50  0000 C CNN
-F 2 "Resistors_THT:R_Axial_DIN0411_L9.9mm_D3.6mm_P15.24mm_Horizontal" V 10430 1150 50  0001 C CNN
+F 2 "Resistors_SMD:R_0805" V 10430 1150 50  0001 C CNN
 F 3 "" H 10500 1150 50  0001 C CNN
 	1    10500 1150
@@
 F 0 "D1" V 2204 6779 50  0000 L CNN
 F 1 "D_Schottky" V 2295 6779 50  0000 L CNN
-F 2 "Diodes_THT:D_DO-41_SOD81_P10.16mm_Horizontal" H 2250 6700 50  0001 C CNN
+F 2 "Diodes_SMD:D_SMA" H 2250 6700 50  0001 C CNN
 F 3 "" H 2250 6700 50  0001 C CNN
 	1    2250 6700
@@
 F 0 "D2" V 2604 6779 50  0000 L CNN
 F 1 "D_Schottky" V 2695 6779 50  0000 L CNN
-F 2 "Diodes_THT:D_DO-41_SOD81_P10.16mm_Horizontal" H 2650 6700 50  0001 C CNN
+F 2 "Diodes_SMD:D_SMA" H 2650 6700 50  0001 C CNN
 F 3 "" H 2650 6700 50  0001 C CNN
 	1    2650 6700
@@
 F 0 "R1" H 2520 6496 50  0000 L CNN
 F 1 "680" H 2520 6405 50  0000 L CNN
-F 2 "Resistors_THT:R_Axial_DIN0204_L3.6mm_D1.6mm_P7.62mm_Horizontal" V 2380 6450 50  0001 C CNN
+F 2 "Resistors_SMD:R_0402" V 2380 6450 50  0001 C CNN
 F 3 "" H 2450 6450 50  0001 C CNN
 	1    2450 6450
@@
 F 0 "C4" V 1998 6200 50  0000 C CNN
 F 1 "10nF" V 2089 6200 50  0000 C CNN
-F 2 "Capacitors_THT:C_Disc_D3.8mm_W2.6mm_P2.50mm" H 2288 6050 50  0001 C CNN
+F 2 "Capacitors_SMD:C_0402" H 2288 6050 50  0001 C CNN
 F 3 "" H 2250 6200 50  0001 C CNN
 	1    2250 6200
@@
 F 0 "C7" H 4268 1146 50  0000 L CNN
 F 1 "4.7uF" H 4268 1055 50  0000 L CNN
-F 2 "Capacitors_THT:CP_Radial_D5.0mm_P2.00mm" H 4188 950 50  0001 C CNN
+F 2 "Capacitors_SMD:CP_Elec_4x5.3" H 4188 950 50  0001 C CNN
 F 3 "" H 4150 1100 50  0001 C CNN
 	1    4150 1100
@@
 F 0 "C12" H 5615 1246 50  0000 L CNN
 F 1 "100nF" H 5615 1155 50  0000 L CNN
-F 2 "Capacitors_THT:C_Disc_D3.8mm_W2.6mm_P2.50mm" H 5538 1050 50  0001 C CNN
+F 2 "Capacitors_SMD:C_0603" H 5538 1050 50  0001 C CNN
 F 3 "" H 5500 1200 50  0001 C CNN
 	1    5500 1200
@@
 F 0 "C17" H 9415 4546 50  0000 L CNN
 F 1 "100nF" H 9415 4455 50  0000 L CNN
-F 2 "Capacitors_THT:C_Disc_D3.8mm_W2.6mm_P2.50mm" H 9338 4350 50  0001 C CNN
+F 2 "Capacitors_SMD:C_0603" H 9338 4350 50  0001 C CNN
 F 3 "" H 9300 4500 50  0001 C CNN
 	1    9300 4500

Commit message: routed everything except for ground
Parts:
- removed Y1: 16MHz, Crystals:Crystal_SMD_SeikoEpson_FA238-4pin_3.2x2.5mm_HandSoldering, symbol device:Crystal
- added J13: RF_Shield_Two_Pieces, Shielding_Cabinets:Laird_Technologies_BMI-S-203-F_26.21x26.21mm, symbol device:RF_Shield_Two_Pieces
- added Y1: 16MHz, Crystals:Crystal_SMD_SeikoEpson_FA238-4pin_3.2x2.5mm, symbol device:Crystal_GND24
- C15: footprint Capacitors_THT:CP_Radial_D5.0mm_P2.00mm -> Capacitors_SMD:CP_Elec_4x5.3
- U4: footprint Housings_DIP:DIP-8_W7.62mm_LongPads -> Housings_SOIC:SOIC-8_3.9x4.9mm_Pitch1.27mm
Connections:
- wire segments 259 -> 262

Commit message: Finished routing ground
Parts:
- U1: footprint TO_SOT_Packages_SMD:TO-252-3_TabPin2 -> TO_SOT_Packages_SMD:TO-252-2
Changed lines of the file:
@@
 F 0 "U1" H 1850 1042 50  0000 C CNN
 F 1 "7805" H 1850 951 50  0000 C CNN
-F 2 "TO_SOT_Packages_SMD:TO-252-3_TabPin2" H 1850 1025 50  0001 C CIN
+F 2 "TO_SOT_Packages_SMD:TO-252-2" H 1850 1025 50  0001 C CIN
 F 3 "http://www.fairchildsemi.com/ds/LM/LM7805.pdf" H 1850 750 50  0001 C CNN
 	1    1850 800
